File: hardware/airwriter/airwriter.kicad_sch (KiCad schematic)
At the start: 56 parts, among them J1 USB-C 5V in, J2 Mini-DIN-8 to printer, J3 Bring-up USB/UART, J4 Mini-DIN-8 LocalTalk, J6 I2C / Qwiic, SW1 BOOT bridge, SW2 MODE/TEST, U1 ESP32-S3-WROOM-1-N8R2, U2 MAX3490ESA+, U3 MAX3232ESE+, U4 AP7361C-33E, U5 USBLC6-2SC6, U6 SP3485EN-L, U7 PIC12F1840-I/P, U8 SP3485EN-L

Commit message: Light the logo with a cavity bounce off three more pixels
Reverse-mount LEDs make a local pool where they sit and do not spread sideways, so
sitting four of them behind a 33mm wordmark would have given four bright patches and
dim gaps between. D4, D5 and D6 are top-firing SK6812MINI instead, shining down into
the printed housing; a white cavity floor bounces the light back up through the
window already diffused, which is what a wide even glow wants.

They sit outside the logo keepout -- (105.5, 93), (146.5, 93), (115, 86.3) -- because
anything under the window would block light coming back up. For a light box the
position barely matters; the cavity floods.

All six pixels are one chain on one wire. U1 IO48 to D1, D1 to D2, then D2's DOUT,
which was hanging unconnected, carries on through D4, D5, D6 over LOGO_CH1/2/3. No
new GPIO, and the logo becomes addressable -- any colour, any animation, same
protocol. Firmware changes one constant from 2 pixels to 6.

SK6812 rather than WS2812B for a real reason found on the way: WS2812B wants 3.5V
minimum and this rail is 3.3V, so the original D1 and D2 were out of spec and nobody
had noticed. Every SK6812 on the board is specified down to 3.3V.

Netlist verified pixel by pixel. ERC is nine lib_symbol_mismatch warnings, all from
symbols flattened into the schematic rather than carried by (extends). DRC is four
violations, all the deliberate cutout removals plus U1. Drill floor 0.300mm.
Parts:
- added D4, D5, D6: SK6812MINI, LED_SMD:LED_SK6812MINI_PLCC4_3.5x3.5mm_P1.75mm, symbol LED:SK6812MINI
Connections:
- net +3V3: now also D4.3 (VDD), D5.3 (VDD), D6.3 (VDD)
- net GND: now also D4.1 (VSS), D5.1 (VSS), D6.1 (VSS)
- net LOGO_CH1: now reaches D2.4 (DOUT)
- net LOGO_CH1: now also D4.2 (DIN)
- new net LOGO_CH2: D4.4 (DOUT), D5.2 (DIN)
- new net LOGO_CH3: D5.4 (DOUT), D6.2 (DIN)
Changed lines of the file:
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@@
     (at 325.12 219.71)
 )
-  (no_connect
-    (at 157.48 223.52)
+  (label "LOGO_CH1"
+    (at 157.48 223.52 0)
+    (effects
+      (font
+        (size 1.27 1.27))
+      (justify left bottom))
 )
   (no_connect
@@
           (unit 1)))))
   (symbol
+    (lib_id "LED:SK6812MINI")
+    (at 33.02 115.57 0)
+    (unit 1)
+    (exclude_from_sim no)
+    (in_bom yes)
+    (on_board yes)
+    (dnp no)
+    (property "Reference" "D4" (at 33.02 104.14 0) (effects (font (size 1.27 1.27))))
+    (property "Value" "SK6812MINI" (at 33.02 127 0) (effects (font (size 1.27 1.27))))
+    (property "Footprint" "LED_SMD:LED_SK6812MINI_PLCC4_3.5x3.5mm_P1.75mm" (at 33.02 115.57 0) (hide yes) (effects (font (size 1.27 1.27))))
+    (property "MPN" "SK6812MINI" (at 33.02 115.57 0) (hide yes) (effects (font (size 1.27 1.27))))
+    (property "Manufacturer" "OPSCO Optoelectronics" (at 33.02 115.57 0) (hide yes) (effects (font (size 1.27 1.27))))
+    (property "Description" "Addressable RGB LED, top firing. Shines down into the housing cavity; the bounce lights the logo window" (at 33.02 115.57 0) (hide yes) (effects (font (size 1.27 1.27))))
+  )
+  (label "+3V3"
+    (at 33.02 107.95 0)
+    (effects
+      (font
+        (size 1.27 1.27))
+      (justify left bottom))
+)
+  (label "GND"
+    (at 33.02 123.19 0)
+    (effects
+      (font
+        (size 1.27 1.27))
+      (justify left bottom))
+)
+  (label "LOGO_CH1"
+    (at 25.4 115.57 0)
+    (effects
+      (font
+        (size 1.27 1.27))
+      (justify left bottom))
+)
+  (label "LOGO_CH2"
+    (at 40.64 115.57 0)
+    (effects
+      (font
+        (size 1.27 1.27))
+      (justify left bottom))
+)
+  (symbol
+    (lib_id "LED:SK6812MINI")
+    (at 54.61 115.57 0)
+    (unit 1)
+    (exclude_from_sim no)
+    (in_bom yes)
+    (on_board yes)
+    (dnp no)
+    (property "Reference" "D5" (at 54.61 104.14 0) (effects (font (size 1.27 1.27))))
+    (property "Value" "SK6812MINI" (at 54.61 127 0) (effects (font (size 1.27 1.27))))
+    (property "Footprint" "LED_SMD:LED_SK6812MINI_PLCC4_3.5x3.5mm_P1.75mm" (at 54.61 115.57 0) (hide yes) (effects (font (size 1.27 1.27))))
+    (property "MPN" "SK6812MINI" (at 54.61 115.57 0) (hide yes) (effects (font (size 1.27 1.27))))
+    (property "Manufacturer" "OPSCO Optoelectronics" (at 54.61 115.57 0) (hide yes) (effects (font (size 1.27 1.27))))
+    (property "Description" "Addressable RGB LED, top firing. Shines down into the housing cavity; the bounce lights the logo window" (at 54.61 115.57 0) (hide yes) (effects (font (size 1.27 1.27))))
+  )
+  (label "+3V3"
+    (at 54.61 107.95 0)
+    (effects
+      (font
+        (size 1.27 1.27))
+      (justify left bottom))
+)
+  (label "GND"
+    (at 54.61 123.19 0)
+    (effects
+      (font
+        (size 1.27 1.27))
+      (justify left bottom))
+)
+  (label "LOGO_CH2"
+    (at 46.99 115.57 0)
+    (effects
+      (font
+        (size 1.27 1.27))
+      (justify left bottom))
+)
+  (label "LOGO_CH3"
+    (at 62.23 115.57 0)
+    (effects
+      (font
+        (size 1.27 1.27))
+      (justify left bottom))
+)
+  (symbol
+    (lib_id "LED:SK6812MINI")
+    (at 77.47 115.57 0)
+    (unit 1)
+    (exclude_from_sim no)
+    (in_bom yes)
+    (on_board yes)
+    (dnp no)
+    (property "Reference" "D6" (at 77.47 104.14 0) (effects (font (size 1.27 1.27))))
+    (property "Value" "SK6812MINI" (at 77.47 127 0) (effects (font (size 1.27 1.27))))
+    (property "Footprint" "LED_SMD:LED_SK6812MINI_PLCC4_3.5x3.5mm_P1.75mm" (at 77.47 115.57 0) (hide yes) (effects (font (size 1.27 1.27))))
+    (property "MPN" "SK6812MINI" (at 77.47 115.57 0) (hide yes) (effects (font (size 1.27 1.27))))
+    (property "Manufacturer" "OPSCO Optoelectronics" (at 77.47 115.57 0) (hide yes) (effects (font (size 1.27 1.27))))
+    (property "Description" "Addressable RGB LED, top firing. Shines down into the housing cavity; the bounce lights the logo window" (at 77.47 115.57 0) (hide yes) (effects (font (size 1.27 1.27))))
+  )
+  (label "+3V3"
+    (at 77.47 107.95 0)
+    (effects
+      (font
+        (size 1.27 1.27))
+      (justify left bottom))
+)
+  (label "GND"
+    (at 77.47 123.19 0)
+    (effects
+      (font
+        (size 1.27 1.27))
+      (justify left bottom))
+)
+  (label "LOGO_CH3"
+    (at 69.85 115.57 0)
+    (effects
+      (font
+        (size 1.27 1.27))
+      (justify left bottom))
+)
+  (no_connect (at 85.09 115.57))
+  (symbol
     (lib_id "Device:R")

Commit message: Make MODE a gold touch pad on the face you actually look at
SW2 stops being a switch. It is now airwriter:TouchPad_Comb_9x7mm -- a comb electrode
on B.Cu with a ground guard bar, mask opened over both so a bare finger meets ENIG
gold on the visible face. The comb is one net; the interleaving is visual. The S3
senses self-capacitance, where a continuous electrode beats an interdigitated one, so
the look costs nothing.

  MODE moves IO38 -> IO14, because the S3 only does touch on IO1-IO14
  R20, 1k, in series: exposed metal on a GPIO is an ESD path and the S3 is rated
    around 2kV while a person carries far more
  C19 goes DNP rather than away -- 100nF across a touch pin would swamp a sense
    capacitance measured in picofarads, and leaving the pads means one part reverts
    MODE to a mechanical switch if touch disappoints

The eurorack precedent is split and worth recording. Make Noise's Rene uses resistive
touch, skin completing a circuit, and is known for not reading on dry hands -- that is
the failure I kept warning about. Synthux's Simple Touch is capacitive via an MPR121
and has no such problem. An MPR121 is twelve channels; overkill for one button when
the S3 has the peripheral built in.

Also corrects an earlier note in the handoff: bare gold is right here. Soldermask is
25 microns and barely matters either way, but exposed ENIG is more sensitive, is what
the synth world does, and is the whole point of paying for the finish.

DRC is four violations, all the deliberate cutout removals plus U1. ERC is nine
lib_symbol_mismatch from flattened symbols. Drill floor 0.300mm, fab regenerated.
Parts:
- added R20: 1k, Resistor_SMD:R_0603_1608Metric, symbol Device:R
- C19: now not fitted
- SW2: value MODE/TEST -> MODE touch; footprint Button_Switch_SMD:SW_SPST_B3U-1000P -> airwriter:TouchPad_Comb_9x7mm; MPN B3U-1000P -> (none); Manufacturer Omron -> none - copper on the board
Connections:
- net BTN_MODE: now also R20.2; no longer U1.31 (IO38)
- net TOUCH_SENSE: now reaches U1.22 (IO14)
- net TOUCH_SENSE: now also R20.1
Changed lines of the file:
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@@
       (justify left bottom))
 )
-  (no_connect
-    (at 189.23 157.48)
+  (label "TOUCH_SENSE"
+    (at 189.23 157.48 0)
+    (effects
+      (font
+        (size 1.27 1.27))
+      (justify left bottom))
 )
   (no_connect
@@
       (xy 222.25 139.7))
 )
-  (wire
-    (pts
-      (xy 219.71 142.24)
-      (xy 222.25 142.24))
-)
   (label "VBUS"
     (at 50.8 44.45 0)
@@
     (at 222.25 139.7 0)
 )
-  (label "BTN_MODE"
-    (at 222.25 142.24 0)
-)
   (symbol
     (lib_id "Connector:USB_C_Receptacle_USB2.0_16P")
@@
         (font
           (size 1.27 1.27))))
-    (property "Value" "MODE/TEST"
+    (property "Value" "MODE touch"
       (at 149.86 199.39 0)
       (effects
         (font
           (size 1.27 1.27))))
-    (property "Footprint" "Button_Switch_SMD:SW_SPST_B3U-1000P"
+    (property "Footprint" "airwriter:TouchPad_Comb_9x7mm"
       (at 149.86 195.58 0)
       (hide yes)
@@
         (font
           (size 1.27 1.27))))
-    (property "MPN" "B3U-1000P"
+    (property "MPN" ""
       (at 149.86 195.58 0)
       (hide yes)
@@
         (font
           (size 1.27 1.27))))
-    (property "Manufacturer" "Omron"
+    (property "Manufacturer" "none - copper on the board"
       (at 149.86 195.58 0)
       (hide yes)
@@
         (font
           (size 1.27 1.27))))
-    (property "Description" "Tactile switch, SMD, 4.8 x 3.4mm"
+    (property "Description" "Capacitive touch pad, exposed gold on the back face. Pad 1 is the electrode, pad 2 the ground guard"
       (at 149.86 195.58 0)
       (hide yes)
@@
     (in_bom yes)
     (on_board yes)
-    (dnp no)
+    (dnp yes)
     (property "Reference" "C19"
       (at 162.56 191.77 0)
@@
       (justify left bottom))
 )
+  (no_connect (at 219.71 142.24))
   (no_connect (at 85.09 115.57))
   (symbol
     (lib_id "Device:R")
+    (at 33.02 133.35 0)
+    (unit 1)
+    (exclude_from_sim no)
+    (in_bom yes)
+    (on_board yes)
+    (dnp no)
+    (property "Reference" "R20" (at 30.48 133.35 90) (effects (font (size 1.27 1.27))))
+    (property "Value" "1k" (at 35.56 133.35 90) (effects (font (size 1.27 1.27))))
+    (property "Footprint" "Resistor_SMD:R_0603_1608Metric" (at 33.02 133.35 0) (hide yes) (effects (font (size 1.27 1.27))))
+    (property "MPN" "" (at 33.02 133.35 0) (hide yes) (effects (font (size 1.27 1.27))))
+    (property "Manufacturer" "Any" (at 33.02 133.35 0) (hide yes) (effects (font (size 1.27 1.27))))
+    (property "Description" "RES 1k 0603. Series ESD limiter between the exposed touch pad and the GPIO" (at 33.02 133.35 0) (hide yes) (effects (font (size 1.27 1.27))))
+  )
+  (label "TOUCH_SENSE"
+    (at 33.02 129.54 0)
+    (effects
+      (font
+        (size 1.27 1.27))
+      (justify left bottom))
+)
+  (label "BTN_MODE"
+    (at 33.02 137.16 0)
+    (effects
+      (font
+        (size 1.27 1.27))
+      (justify left bottom))
+)
+  (symbol
+    (lib_id "Device:R")

Commit message: Put the touch pattern in the soldermask instead of the copper
The comb was chunky and, worse, it cut the electrode up. Self-capacitance wants
unbroken area, so carving the copper into fingers or a halftone trades sensitivity
for looks.

So the copper does not carry the pattern at all. The electrode is a solid 9.2mm disc
and the mask opens along eleven thin arcs, 0.18mm wide on a 0.45mm pitch, rotating
and lengthening as the radius grows so it reads as a ripple rather than a bullseye.
What you see is fine gold arcs on matte black; what the chip sees is a full disc.
Same trick as the logo -- mask carries the artwork, copper carries the function.

First attempt packed the arcs on a 0.265mm pitch, which left 0.045mm mask dams. That
is under half PCBWay's 0.1mm floor and would have flooded into one solid blob. At
0.45mm pitch the dams are 0.27mm, comfortably clear.

The footprint is generated, not drawn -- TouchPad_Arcs_D9mm.kicad_mod comes out of a
short script, so the rhythm can be re-cut by changing three numbers.

DRC still four violations, all the deliberate cutout removals plus U1. Drill floor
0.300mm, 18 mask apertures on the back layer, fab regenerated.
Parts:
- SW2: footprint airwriter:TouchPad_Comb_9x7mm -> airwriter:TouchPad_Arcs_D9mm
Changed lines of the file:
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@@
         (font
           (size 1.27 1.27))))
-    (property "Footprint" "airwriter:TouchPad_Comb_9x7mm"
+    (property "Footprint" "airwriter:TouchPad_Arcs_D9mm"
       (at 149.86 195.58 0)
       (hide yes)
@@
         (font
           (size 1.27 1.27))))
-    (property "Description" "Capacitive touch pad, exposed gold on the back face. Pad 1 is the electrode, pad 2 the ground guard"
+    (property "Description" "Capacitive touch pad on the back face. Solid copper disc with the pattern in the soldermask, so it reads as fine gold arcs on black"
       (at 149.86 195.58 0)
       (hide yes)

Commit message: Drop the credit line and turn BOOT into a bullseye you can reach
The TashTalk credit ran the full width of B.Silkscreen and was eating a band of the
grain -- silk over exposed copper does not adhere, so every artwork cell beneath it
had to give way, 141 of them. The attribution still stands in the handoff, in SPEC.md
and in the licence; it does not need to be on the show face.

SW1 was SolderJumper-2_Open on the component side, which is inside the case. You
would have had to open the housing to reach a pad whose entire purpose is insurance
when USB will not enumerate. It is now airwriter:BootPads_Ring_D5mm on the back: a
2.2mm disc inside a 0.9mm ring, 0.5mm apart, both exposed ENIG. Bridge with tweezers.
Ø5mm against the MODE pad's Ø9.2mm so it reads as the secondary control, and the
concentric geometry answers MODE's arcs rather than fighting them.

artwork.py now carries the import, so the artwork is reproducible rather than a
one-off. It filters every cell against the copper actually on the board and emits
rule areas barring copper pour only, so it never forces a re-route. The order it
depends on is documented: strip, route, stitch, prune vias, artwork, refill.

Retention improved with the credit gone: wordmark FR4 280, grain 22, gold 776.

DRC is four, all the deliberate footprint mismatches. Drill floor 0.300mm.
Parts:
- SW1: footprint Jumper:SolderJumper-2_P1.3mm_Open_Pad1.0x1.5mm -> airwriter:BootPads_Ring_D5mm
Changed lines of the file:
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@@
         (font
           (size 1.27 1.27))))
-    (property "Footprint" "Jumper:SolderJumper-2_P1.3mm_Open_Pad1.0x1.5mm"
+    (property "Footprint" "airwriter:BootPads_Ring_D5mm"
       (at 149.86 175.26 0)
       (hide yes)
@@
         (font
           (size 1.27 1.27))))
-    (property "Description" "Two exposed pads, normally open. Bridge with tweezers to force download mode; the USB-C port normally does this without them"
+    (property "Description" "BOOT bridge on the back face: a gold disc inside a gold ring, 0.5mm apart. Short with tweezers to force download mode; the USB-C port normally does this without them"
       (at 149.86 171.45 0)
       (hide yes)

Commit message: Dither the two touch controls onto the cover's grid
The arcs and the bullseye were the only smooth geometry on a board whose whole back
is a dithered wordmark dissolving into grain. They read as hardware dropped onto the
artwork rather than as part of it.

Both are dithered now, on the cover's own 0.455mm cell grid, with density falling off
by radius. That fade is what makes a flat field read as a target instead of a blob,
and it echoes the way the grain dissolves above and below the wordmark. MODE is 150
cells over its 9.2mm disc; BOOT is a dense core inside a dithered ring at half the
diameter, so it still reads as the secondary control.

The copper did not change -- same solid disc for MODE, same disc-and-ring for BOOT --
so nothing needed re-routing. Only the soldermask moved, which is the same principle
the logo and the artwork already run on: mask carries the picture, copper carries the
function.

Both footprints come out of lib/gen_touchpads.py now, so grid, cell size and the
density curve are three numbers in one place rather than hand-drawn geometry. The
superseded arc and ring footprints are deleted.

DRC is four, all the deliberate footprint mismatches. Drill floor 0.300mm, 1258 mask
apertures on the back.
Parts:
- SW1: footprint airwriter:BootPads_Ring_D5mm -> airwriter:BootPads_Dither_D5mm
- SW2: footprint airwriter:TouchPad_Arcs_D9mm -> airwriter:TouchPad_Dither_D9mm
Changed lines of the file:
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@@
         (font
           (size 1.27 1.27))))
-    (property "Footprint" "airwriter:BootPads_Ring_D5mm"
+    (property "Footprint" "airwriter:BootPads_Dither_D5mm"
       (at 149.86 175.26 0)
       (hide yes)
@@
         (font
           (size 1.27 1.27))))
-    (property "Description" "BOOT bridge on the back face: a gold disc inside a gold ring, 0.5mm apart. Short with tweezers to force download mode; the USB-C port normally does this without them"
+    (property "Description" "BOOT bridge, back face: a dithered disc inside a dithered ring, 0.5mm apart. Short with tweezers to force download mode"
       (at 149.86 171.45 0)
       (hide yes)
@@
         (font
           (size 1.27 1.27))))
-    (property "Footprint" "airwriter:TouchPad_Arcs_D9mm"
+    (property "Footprint" "airwriter:TouchPad_Dither_D9mm"
       (at 149.86 195.58 0)
       (hide yes)
@@
         (font
           (size 1.27 1.27))))
-    (property "Description" "Capacitive touch pad on the back face. Solid copper disc with the pattern in the soldermask, so it reads as fine gold arcs on black"
+    (property "Description" "Capacitive touch pad, back face. Solid copper disc with a dithered mask on the cover artwork grid, fading outward"
       (at 149.86 195.58 0)
       (hide yes)

Commit message: Redraw MODE in the mist's own cells and demote BOOT to a service point
Wells read the fine dither on SW2 as a clump that matched neither logo
nor mist. The pad keeps its solid 9.2mm electrode; the mask now draws a
solid gold core dissolving outward in the grain's 0.72mm cells, so the
control reads as the mist condensing.

SW1 stops posing as a button. It moves to the component side as two
plain labelled pads on the same coordinates -- the F.Cu track lands on
pad 1 unchanged -- and loses its through-hole, so the visible face
carries exactly one control. Mist backfills where its bullseye sat.

D4-D6 pointed at a 3D model KiCad 10 does not ship and rendered as
empty pads; they borrow the WS2812B-Mini step, the same 3.5mm PLCC4.

ERC clean. DRC: 0 violations, the same 11 pre-existing pour-fragment
notes as before the change.
Parts:
- SW1: footprint airwriter:BootPads_Dither_D5mm -> airwriter:BootPads_Service
- SW2: footprint airwriter:TouchPad_Dither_D9mm -> airwriter:TouchPad_Core_D9mm
Changed lines of the file:
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@@
         (font
           (size 1.27 1.27))))
-    (property "Footprint" "airwriter:BootPads_Dither_D5mm"
+    (property "Footprint" "airwriter:BootPads_Service"
       (at 149.86 175.26 0)
       (hide yes)
@@
         (font
           (size 1.27 1.27))))
-    (property "Footprint" "airwriter:TouchPad_Dither_D9mm"
+    (property "Footprint" "airwriter:TouchPad_Core_D9mm"
       (at 149.86 195.58 0)
       (hide yes)
