File: hardware/panel/panel.kicad_pcb (KiCad board)
At the start: 2 copper layers, 62 x 104.3 mm, 5 parts

Commit message: Panel: close mask to the copper edge around the test hole — no FR4 sliver
The marker circle (3.83mm) sits inside the hole-clearance floor (copper
can't start before 4.4mm), so keeping mask closed only to the marker left
a 0.3mm bare-FR4 ring. Mask now closes to max(marker, hole+0.6): the black
ring runs from drill to gold with nothing between.
Parts:
- moved MT2 100.1 mm to (56.4, 5.64)
- moved MT3 100.1 mm to (5.64, 91.9)
- moved MT1 98.6 mm to (5.64, 5.64)
- moved MT4 98.6 mm to (53.4, 91.9)
- renumbered MT4 to MT1, MT3 to MT2, MT2 to MT3, MT1 to MT4
Changed lines of the file:
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@@
 	(footprint "panel:SMT_Standoff_M2.5_D6.0mm"
 		(layer "B.Cu")
-		(at 53.3636 91.93)
-		(property "Reference" "MT4"
+		(at 5.6364 5.6364)
+		(property "Reference" "MT1"
 			(at 0 0 0)
 			(layer "F.SilkS")
@@
 	(footprint "panel:SMT_Standoff_M2.5_D6.0mm"
 		(layer "B.Cu")
-		(at 5.6364 5.6364)
-		(property "Reference" "MT1"
+		(at 53.3636 91.93)
+		(property "Reference" "MT4"
 			(at 0 0 0)
 			(layer "F.SilkS")
@@
 	(footprint "panel:SMT_Standoff_M2.5_D6.0mm"
 		(layer "B.Cu")
-		(at 5.6364 91.93)
-		(property "Reference" "MT3"
+		(at 56.3636 5.6364)
+		(property "Reference" "MT2"
 			(at 0 0 0)
 			(layer "F.SilkS")
@@
 	(footprint "panel:SMT_Standoff_M2.5_D6.0mm"
 		(layer "B.Cu")
-		(at 56.3636 5.6364)
-		(property "Reference" "MT2"
+		(at 5.6364 91.93)
+		(property "Reference" "MT3"
 			(at 0 0 0)
 			(layer "F.SilkS")
@@
 			(xy 31.925 33.1743) (xy 31.8576 33.4039) (xy 31.8425 33.6833) (xy 31.84527 33.687119) (xy 31.81808 33.696849)
 			(xy 31.765518 33.710015) (xy 31.7522 33.7115) (xy 31.7307 33.714) (xy 31.7167 33.715) (xy 31.6317 33.6951)
-			(xy 31.6088 33.6477) (xy 31.6152 33.5916) (xy 31.6524 33.4174) (xy 31.6896 33.243299) (xy 31.7268 33.0691)
-			(xy 31.7888 33.0691) (xy 31.8508 33.0691) (xy 31.9128 33.0691) (xy 31.9201 33.0342) (xy 31.9275 32.9992)
-			(xy 31.9348 32.9643) (xy 31.8728 32.9643) (xy 31.8108 32.9643) (xy 31.7488 32.9643) (xy 31.7651 32.8887)
-			(xy 31.7815 32.8132) (xy 31.797606 32.738595) (xy 31.902724 32.688879) (xy 32.063916 32.592264) (xy 32.214863 32.480315)
-			(xy 32.354109 32.354109) (xy 32.480315 32.214863) (xy 32.592264 32.063916) (xy 32.688879 31.902724)
-			(xy 32.769229 31.732838) (xy 32.83254 31.555895) (xy 32.878203 31.373597) (xy 32.905778 31.187702)
-			(xy 32.915 31) (xy 32.905778 30.812297) (xy 32.878203 30.626402) (xy 32.83254 30.444104) (xy 32.769229 30.267161)
-			(xy 32.688879 30.097275) (xy 32.592264 29.936083) (xy 32.480315 29.785136) (xy 32.354109 29.64589)
-			(xy 32.214863 29.519684) (xy 32.063916 29.407735) (xy 31.902724 29.31112) (xy 31.732838 29.23077)
-			(xy 31.555895 29.167459) (xy 31.373597 29.121796) (xy 31.187702 29.094221) (xy 31 29.085) (xy 30.812297 29.094221)
-			(xy 30.626402 29.121796) (xy 30.444104 29.167459) (xy 30.267161 29.23077) (xy 30.097275 29.31112)
-			(xy 29.936083 29.407735) (xy 29.785136 29.519684) (xy 29.64589 29.64589) (xy 29.519684 29.785136)
-			(xy 29.407735 29.936083) (xy 29.31112 30.097275) (xy 29.23077 30.267161) (xy 29.167459 30.444104)
-			(xy 29.121796 30.626402) (xy 29.094221 30.812297) (xy 29.085 31) (xy 29.094221 31.187702) (xy 29.121796 31.373597)
-			(xy 29.167459 31.555895) (xy 29.23077 31.732838) (xy 29.31112 31.902724) (xy 29.407735 32.063916)
-			(xy 29.519684 32.214863) (xy 29.64589 32.354109) (xy 29.785136 32.480315) (xy 29.936083 32.592264)
-			(xy 30.097275 32.688879) (xy 30.267161 32.769229) (xy 30.444104 32.83254) (xy 30.626402 32.878203)
-			(xy 30.812297 32.905778) (xy 31 32.915) (xy 31.187702 32.905778) (xy 31.373597 32.878203) (xy 31.555895 32.83254)
-			(xy 31.645566 32.800455) (xy 31.6338 32.8549) (xy 31.622 32.909599) (xy 31.6101 32.9643) (xy 31.5634 32.9643)
-			(xy 31.5166 32.9643) (xy 31.4698 32.9643) (xy 31.4625 32.9992) (xy 31.4551 33.0342) (xy 31.4478 33.0691)
-			(xy 31.4946 33.0691) (xy 31.5414 33.0691) (xy 31.5882 33.0691) (xy 31.5453 33.2715) (xy 31.5025 33.473799)
-			(xy 31.4596 33.6761) (xy 31.4625 33.7592) (xy 31.478078 33.774688) (xy 31.276231 33.804629) (xy 31 33.8182)
-			(xy 30.723768 33.804629) (xy 30.450196 33.764049) (xy 30.181919 33.696849) (xy 29.921521 33.603677)
-			(xy 29.671509 33.48543) (xy 29.434291 33.343247) (xy 29.212152 33.178498) (xy 29.007231 32.992768)
-			(xy 28.821501 32.787847) (xy 28.656752 32.565708) (xy 28.514569 32.32849) (xy 28.396322 32.078478)
-			(xy 28.30315 31.81808) (xy 28.23595 31.549803) (xy 28.19537 31.276231) (xy 28.1818 31) (xy 28.19537 30.723768)
-			(xy 28.23595 30.450196) (xy 28.30315 30.181919) (xy 28.396322 29.921521) (xy 28.514569 29.671509)
-			(xy 28.656752 29.434291) (xy 28.821501 29.212152) (xy 29.007231 29.007231) (xy 29.212152 28.821501)
-			(xy 29.434291 28.656752) (xy 29.671509 28.514569) (xy 29.921521 28.396322) (xy 30.181919 28.30315)
-			(xy 30.450196 28.23595) (xy 30.723768 28.19537) (xy 31 28.1818)
+			(xy 31.6088 33.6477) (xy 31.6152 33.5916) (xy 31.6524 33.4174) (xy 31.6896 33.243299) (xy 31.725732 33.0741)
+			(xy 31.739708 33.0691) (xy 31.7888 33.0691) (xy 31.8508 33.0691) (xy 31.9128 33.0691) (xy 31.9201 33.0342)
+			(xy 31.9275 32.9992) (xy 31.929159 32.991264) (xy 32.037072 32.940226) (xy 32.222254 32.829233) (xy 32.395665 32.700622)
+			(xy 32.555634 32.555634) (xy 32.700622 32.395665) (xy 32.829233 32.222254) (xy 32.940226 32.037072)
+			(xy 33.032534 31.841903) (xy 33.105268 31.638626) (xy 33.157727 31.429198) (xy 33.189406 31.215637)
+			(xy 33.2 31) (xy 33.189406 30.784362) (xy 33.157727 30.570801) (xy 33.105268 30.361373) (xy 33.032534 30.158096)
+			(xy 32.940226 29.962927) (xy 32.829233 29.777745) (xy 32.700622 29.604334) (xy 32.555634 29.444365)
+			(xy 32.395665 29.299377) (xy 32.222254 29.170766) (xy 32.037072 29.059773) (xy 31.841903 28.967465)
+			(xy 31.638626 28.894731) (xy 31.429198 28.842272) (xy 31.215637 28.810593) (xy 31 28.8) (xy 30.784362 28.810593)
+			(xy 30.570801 28.842272) (xy 30.361373 28.894731) (xy 30.158096 28.967465) (xy 29.962927 29.059773)
+			(xy 29.777745 29.170766) (xy 29.604334 29.299377) (xy 29.444365 29.444365) (xy 29.299377 29.604334)
+			(xy 29.170766 29.777745) (xy 29.059773 29.962927) (xy 28.967465 30.158096) (xy 28.894731 30.361373)
+			(xy 28.842272 30.570801) (xy 28.810593 30.784362) (xy 28.8 31) (xy 28.810593 31.215637) (xy 28.842272 31.429198)
+			(xy 28.894731 31.638626) (xy 28.967465 31.841903) (xy 29.059773 32.037072) (xy 29.170766 32.222254)
+			(xy 29.299377 32.395665) (xy 29.444365 32.555634) (xy 29.604334 32.700622) (xy 29.777745 32.829233)
+			(xy 29.962927 32.940226) (xy 30.158096 33.032534) (xy 30.361373 33.105268) (xy 30.570801 33.157727)
+			(xy 30.784362 33.189406) (xy 31 33.2) (xy 31.215637 33.189406) (xy 31.429198 33.157727) (xy 31.577276 33.120635)
+			(xy 31.5453 33.2715) (xy 31.5025 33.473799) (xy 31.4596 33.6761) (xy 31.4625 33.7592) (xy 31.478078 33.774688)
+			(xy 31.276231 33.804629) (xy 31 33.8182) (xy 30.723768 33.804629) (xy 30.450196 33.764049) (xy 30.181919 33.696849)
+			(xy 29.921521 33.603677) (xy 29.671509 33.48543) (xy 29.434291 33.343247) (xy 29.212152 33.178498)
+			(xy 29.007231 32.992768) (xy 28.821501 32.787847) (xy 28.656752 32.565708) (xy 28.514569 32.32849)
+			(xy 28.396322 32.078478) (xy 28.30315 31.81808) (xy 28.23595 31.549803) (xy 28.19537 31.276231) (xy 28.1818 31)
+			(xy 28.19537 30.723768) (xy 28.23595 30.450196) (xy 28.30315 30.181919) (xy 28.396322 29.921521)
+			(xy 28.514569 29.671509) (xy 28.656752 29.434291) (xy 28.821501 29.212152) (xy 29.007231 29.007231)
+			(xy 29.212152 28.821501) (xy 29.434291 28.656752) (xy 29.671509 28.514569) (xy 29.921521 28.396322)
+			(xy 30.181919 28.30315) (xy 30.450196 28.23595) (xy 30.723768 28.19537) (xy 31 28.1818)
 		)
 		(stroke
