File: hardware/combined/panel-flipped.kicad_pcb (KiCad board)
At the start: 2 copper layers, 62 x 104.3 mm, 5 parts

Commit message: Panel: close mask to the copper edge around the test hole — no FR4 sliver
The marker circle (3.83mm) sits inside the hole-clearance floor (copper
can't start before 4.4mm), so keeping mask closed only to the marker left
a 0.3mm bare-FR4 ring. Mask now closes to max(marker, hole+0.6): the black
ring runs from drill to gold with nothing between.
Parts:
- moved MT2 100.1 mm to (5.64, 5.64)
- moved MT3 100.1 mm to (56.4, 91.9)
- moved MT1 98.6 mm to (56.4, 5.64)
- moved MT4 98.6 mm to (8.64, 91.9)
- renumbered MT4 to MT1, MT3 to MT2, MT2 to MT3, MT1 to MT4
Changed lines of the file:
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@@
 	(footprint "panel:SMT_Standoff_M2.5_D6.0mm"
 		(layer "F.Cu")
-		(at 5.6364 5.6364 180)
-		(property "Reference" "MT2"
+		(at 56.3636 91.93 180)
+		(property "Reference" "MT3"
 			(at 0 0 0)
 			(layer "B.SilkS")
@@
 	(footprint "panel:SMT_Standoff_M2.5_D6.0mm"
 		(layer "F.Cu")
-		(at 56.3636 5.6364 180)
-		(property "Reference" "MT1"
+		(at 8.6364 91.93 180)
+		(property "Reference" "MT4"
 			(at 0 0 0)
 			(layer "B.SilkS")
@@
 	(footprint "panel:SMT_Standoff_M2.5_D6.0mm"
 		(layer "F.Cu")
-		(at 8.6364 91.93 180)
-		(property "Reference" "MT4"
+		(at 56.3636 5.6364 180)
+		(property "Reference" "MT1"
 			(at 0 0 0)
 			(layer "B.SilkS")
@@
 	(footprint "panel:SMT_Standoff_M2.5_D6.0mm"
 		(layer "F.Cu")
-		(at 56.3636 91.93 180)
-		(property "Reference" "MT3"
+		(at 5.6364 5.6364 180)
+		(property "Reference" "MT2"
 			(at 0 0 0)
 			(layer "B.SilkS")
@@
 			(xy 30.075 33.1743) (xy 30.1424 33.4039) (xy 30.1575 33.6833) (xy 30.15473 33.687119) (xy 30.18192 33.696849)
 			(xy 30.234482 33.710015) (xy 30.2478 33.7115) (xy 30.2693 33.714) (xy 30.2833 33.715) (xy 30.3683 33.6951)
-			(xy 30.3912 33.6477) (xy 30.3848 33.5916) (xy 30.3476 33.4174) (xy 30.3104 33.243299) (xy 30.2732 33.0691)
-			(xy 30.2112 33.0691) (xy 30.1492 33.0691) (xy 30.0872 33.0691) (xy 30.0799 33.0342) (xy 30.0725 32.9992)
-			(xy 30.0652 32.9643) (xy 30.1272 32.9643) (xy 30.1892 32.9643) (xy 30.2512 32.9643) (xy 30.2349 32.8887)
-			(xy 30.2185 32.8132) (xy 30.202394 32.738595) (xy 30.097276 32.688879) (xy 29.936084 32.592264) (xy 29.785137 32.480315)
-			(xy 29.645891 32.354109) (xy 29.519685 32.214863) (xy 29.407736 32.063916) (xy 29.311121 31.902724)
-			(xy 29.230771 31.732838) (xy 29.16746 31.555895) (xy 29.121797 31.373597) (xy 29.094222 31.187702)
-			(xy 29.085 31) (xy 29.094222 30.812297) (xy 29.121797 30.626402) (xy 29.16746 30.444104) (xy 29.230771 30.267161)
-			(xy 29.311121 30.097275) (xy 29.407736 29.936083) (xy 29.519685 29.785136) (xy 29.645891 29.64589)
-			(xy 29.785137 29.519684) (xy 29.936084 29.407735) (xy 30.097276 29.31112) (xy 30.267162 29.23077)
-			(xy 30.444105 29.167459) (xy 30.626403 29.121796) (xy 30.812298 29.094221) (xy 31 29.085) (xy 31.187703 29.094221)
-			(xy 31.373598 29.121796) (xy 31.555896 29.167459) (xy 31.732839 29.23077) (xy 31.902725 29.31112)
-			(xy 32.063917 29.407735) (xy 32.214864 29.519684) (xy 32.35411 29.64589) (xy 32.480316 29.785136)
-			(xy 32.592265 29.936083) (xy 32.68888 30.097275) (xy 32.76923 30.267161) (xy 32.832541 30.444104)
-			(xy 32.878204 30.626402) (xy 32.905779 30.812297) (xy 32.915 31) (xy 32.905779 31.187702) (xy 32.878204 31.373597)
-			(xy 32.832541 31.555895) (xy 32.76923 31.732838) (xy 32.68888 31.902724) (xy 32.592265 32.063916)
-			(xy 32.480316 32.214863) (xy 32.35411 32.354109) (xy 32.214864 32.480315) (xy 32.063917 32.592264)
-			(xy 31.902725 32.688879) (xy 31.732839 32.769229) (xy 31.555896 32.83254) (xy 31.373598 32.878203)
-			(xy 31.187703 32.905778) (xy 31 32.915) (xy 30.812298 32.905778) (xy 30.626403 32.878203) (xy 30.444105 32.83254)
-			(xy 30.354434 32.800455) (xy 30.3662 32.8549) (xy 30.378 32.909599) (xy 30.3899 32.9643) (xy 30.4366 32.9643)
-			(xy 30.4834 32.9643) (xy 30.5302 32.9643) (xy 30.5375 32.9992) (xy 30.5449 33.0342) (xy 30.5522 33.0691)
-			(xy 30.5054 33.0691) (xy 30.4586 33.0691) (xy 30.4118 33.0691) (xy 30.4547 33.2715) (xy 30.4975 33.473799)
-			(xy 30.5404 33.6761) (xy 30.5375 33.7592) (xy 30.521922 33.774688) (xy 30.723769 33.804629) (xy 31 33.8182)
-			(xy 31.276232 33.804629) (xy 31.549804 33.764049) (xy 31.818081 33.696849) (xy 32.078479 33.603677)
-			(xy 32.328491 33.48543) (xy 32.565709 33.343247) (xy 32.787848 33.178498) (xy 32.992769 32.992768)
-			(xy 33.178499 32.787847) (xy 33.343248 32.565708) (xy 33.485431 32.32849) (xy 33.603678 32.078478)
-			(xy 33.69685 31.81808) (xy 33.76405 31.549803) (xy 33.80463 31.276231) (xy 33.8182 31) (xy 33.80463 30.723768)
-			(xy 33.76405 30.450196) (xy 33.69685 30.181919) (xy 33.603678 29.921521) (xy 33.485431 29.671509)
-			(xy 33.343248 29.434291) (xy 33.178499 29.212152) (xy 32.992769 29.007231) (xy 32.787848 28.821501)
-			(xy 32.565709 28.656752) (xy 32.328491 28.514569) (xy 32.078479 28.396322) (xy 31.818081 28.30315)
-			(xy 31.549804 28.23595) (xy 31.276232 28.19537) (xy 31 28.1818)
+			(xy 30.3912 33.6477) (xy 30.3848 33.5916) (xy 30.3476 33.4174) (xy 30.3104 33.243299) (xy 30.274268 33.0741)
+			(xy 30.260292 33.0691) (xy 30.2112 33.0691) (xy 30.1492 33.0691) (xy 30.0872 33.0691) (xy 30.0799 33.0342)
+			(xy 30.0725 32.9992) (xy 30.070841 32.991264) (xy 29.962928 32.940226) (xy 29.777746 32.829233) (xy 29.604335 32.700622)
+			(xy 29.444366 32.555634) (xy 29.299378 32.395665) (xy 29.170767 32.222254) (xy 29.059774 32.037072)
+			(xy 28.967466 31.841903) (xy 28.894732 31.638626) (xy 28.842273 31.429198) (xy 28.810594 31.215637)
+			(xy 28.8 31) (xy 28.810594 30.784362) (xy 28.842273 30.570801) (xy 28.894732 30.361373) (xy 28.967466 30.158096)
+			(xy 29.059774 29.962927) (xy 29.170767 29.777745) (xy 29.299378 29.604334) (xy 29.444366 29.444365)
+			(xy 29.604335 29.299377) (xy 29.777746 29.170766) (xy 29.962928 29.059773) (xy 30.158097 28.967465)
+			(xy 30.361374 28.894731) (xy 30.570802 28.842272) (xy 30.784363 28.810593) (xy 31 28.8) (xy 31.215638 28.810593)
+			(xy 31.429199 28.842272) (xy 31.638627 28.894731) (xy 31.841904 28.967465) (xy 32.037073 29.059773)
+			(xy 32.222255 29.170766) (xy 32.395666 29.299377) (xy 32.555635 29.444365) (xy 32.700623 29.604334)
+			(xy 32.829234 29.777745) (xy 32.940227 29.962927) (xy 33.032535 30.158096) (xy 33.105269 30.361373)
+			(xy 33.157728 30.570801) (xy 33.189407 30.784362) (xy 33.2 31) (xy 33.189407 31.215637) (xy 33.157728 31.429198)
+			(xy 33.105269 31.638626) (xy 33.032535 31.841903) (xy 32.940227 32.037072) (xy 32.829234 32.222254)
+			(xy 32.700623 32.395665) (xy 32.555635 32.555634) (xy 32.395666 32.700622) (xy 32.222255 32.829233)
+			(xy 32.037073 32.940226) (xy 31.841904 33.032534) (xy 31.638627 33.105268) (xy 31.429199 33.157727)
+			(xy 31.215638 33.189406) (xy 31 33.2) (xy 30.784363 33.189406) (xy 30.570802 33.157727) (xy 30.422724 33.120635)
+			(xy 30.4547 33.2715) (xy 30.4975 33.473799) (xy 30.5404 33.6761) (xy 30.5375 33.7592) (xy 30.521922 33.774688)
+			(xy 30.723769 33.804629) (xy 31 33.8182) (xy 31.276232 33.804629) (xy 31.549804 33.764049) (xy 31.818081 33.696849)
+			(xy 32.078479 33.603677) (xy 32.328491 33.48543) (xy 32.565709 33.343247) (xy 32.787848 33.178498)
+			(xy 32.992769 32.992768) (xy 33.178499 32.787847) (xy 33.343248 32.565708) (xy 33.485431 32.32849)
+			(xy 33.603678 32.078478) (xy 33.69685 31.81808) (xy 33.76405 31.549803) (xy 33.80463 31.276231) (xy 33.8182 31)
+			(xy 33.80463 30.723768) (xy 33.76405 30.450196) (xy 33.69685 30.181919) (xy 33.603678 29.921521)
+			(xy 33.485431 29.671509) (xy 33.343248 29.434291) (xy 33.178499 29.212152) (xy 32.992769 29.007231)
+			(xy 32.787848 28.821501) (xy 32.565709 28.656752) (xy 32.328491 28.514569) (xy 32.078479 28.396322)
+			(xy 31.818081 28.30315) (xy 31.549804 28.23595) (xy 31.276232 28.19537) (xy 31 28.1818)
 		)
 		(stroke

Commit message: Revert "Panel: close mask to the copper edge around the test hole — no FR4 sliver"
This reverts commit eb9a4d2783863aab7f219a44ac207152b572bd98.
Parts:
- moved MT2 100.1 mm to (5.64, 5.64)
- moved MT3 100.1 mm to (56.4, 91.9)
- moved MT1 98.6 mm to (56.4, 5.64)
- moved MT4 98.6 mm to (8.64, 91.9)
- renumbered MT4 to MT1, MT3 to MT2, MT2 to MT3, MT1 to MT4
Changed lines of the file:
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@@
 	(footprint "panel:SMT_Standoff_M2.5_D6.0mm"
 		(layer "F.Cu")
-		(at 56.3636 91.93 180)
-		(property "Reference" "MT3"
+		(at 5.6364 5.6364 180)
+		(property "Reference" "MT2"
 			(at 0 0 0)
 			(layer "B.SilkS")
@@
 	(footprint "panel:SMT_Standoff_M2.5_D6.0mm"
 		(layer "F.Cu")
-		(at 8.6364 91.93 180)
-		(property "Reference" "MT4"
+		(at 56.3636 5.6364 180)
+		(property "Reference" "MT1"
 			(at 0 0 0)
 			(layer "B.SilkS")
@@
 	(footprint "panel:SMT_Standoff_M2.5_D6.0mm"
 		(layer "F.Cu")
-		(at 56.3636 5.6364 180)
-		(property "Reference" "MT1"
+		(at 8.6364 91.93 180)
+		(property "Reference" "MT4"
 			(at 0 0 0)
 			(layer "B.SilkS")
@@
 	(footprint "panel:SMT_Standoff_M2.5_D6.0mm"
 		(layer "F.Cu")
-		(at 5.6364 5.6364 180)
-		(property "Reference" "MT2"
+		(at 56.3636 91.93 180)
+		(property "Reference" "MT3"
 			(at 0 0 0)
 			(layer "B.SilkS")
@@
 			(xy 30.075 33.1743) (xy 30.1424 33.4039) (xy 30.1575 33.6833) (xy 30.15473 33.687119) (xy 30.18192 33.696849)
 			(xy 30.234482 33.710015) (xy 30.2478 33.7115) (xy 30.2693 33.714) (xy 30.2833 33.715) (xy 30.3683 33.6951)
-			(xy 30.3912 33.6477) (xy 30.3848 33.5916) (xy 30.3476 33.4174) (xy 30.3104 33.243299) (xy 30.274268 33.0741)
-			(xy 30.260292 33.0691) (xy 30.2112 33.0691) (xy 30.1492 33.0691) (xy 30.0872 33.0691) (xy 30.0799 33.0342)
-			(xy 30.0725 32.9992) (xy 30.070841 32.991264) (xy 29.962928 32.940226) (xy 29.777746 32.829233) (xy 29.604335 32.700622)
-			(xy 29.444366 32.555634) (xy 29.299378 32.395665) (xy 29.170767 32.222254) (xy 29.059774 32.037072)
-			(xy 28.967466 31.841903) (xy 28.894732 31.638626) (xy 28.842273 31.429198) (xy 28.810594 31.215637)
-			(xy 28.8 31) (xy 28.810594 30.784362) (xy 28.842273 30.570801) (xy 28.894732 30.361373) (xy 28.967466 30.158096)
-			(xy 29.059774 29.962927) (xy 29.170767 29.777745) (xy 29.299378 29.604334) (xy 29.444366 29.444365)
-			(xy 29.604335 29.299377) (xy 29.777746 29.170766) (xy 29.962928 29.059773) (xy 30.158097 28.967465)
-			(xy 30.361374 28.894731) (xy 30.570802 28.842272) (xy 30.784363 28.810593) (xy 31 28.8) (xy 31.215638 28.810593)
-			(xy 31.429199 28.842272) (xy 31.638627 28.894731) (xy 31.841904 28.967465) (xy 32.037073 29.059773)
-			(xy 32.222255 29.170766) (xy 32.395666 29.299377) (xy 32.555635 29.444365) (xy 32.700623 29.604334)
-			(xy 32.829234 29.777745) (xy 32.940227 29.962927) (xy 33.032535 30.158096) (xy 33.105269 30.361373)
-			(xy 33.157728 30.570801) (xy 33.189407 30.784362) (xy 33.2 31) (xy 33.189407 31.215637) (xy 33.157728 31.429198)
-			(xy 33.105269 31.638626) (xy 33.032535 31.841903) (xy 32.940227 32.037072) (xy 32.829234 32.222254)
-			(xy 32.700623 32.395665) (xy 32.555635 32.555634) (xy 32.395666 32.700622) (xy 32.222255 32.829233)
-			(xy 32.037073 32.940226) (xy 31.841904 33.032534) (xy 31.638627 33.105268) (xy 31.429199 33.157727)
-			(xy 31.215638 33.189406) (xy 31 33.2) (xy 30.784363 33.189406) (xy 30.570802 33.157727) (xy 30.422724 33.120635)
-			(xy 30.4547 33.2715) (xy 30.4975 33.473799) (xy 30.5404 33.6761) (xy 30.5375 33.7592) (xy 30.521922 33.774688)
-			(xy 30.723769 33.804629) (xy 31 33.8182) (xy 31.276232 33.804629) (xy 31.549804 33.764049) (xy 31.818081 33.696849)
-			(xy 32.078479 33.603677) (xy 32.328491 33.48543) (xy 32.565709 33.343247) (xy 32.787848 33.178498)
-			(xy 32.992769 32.992768) (xy 33.178499 32.787847) (xy 33.343248 32.565708) (xy 33.485431 32.32849)
-			(xy 33.603678 32.078478) (xy 33.69685 31.81808) (xy 33.76405 31.549803) (xy 33.80463 31.276231) (xy 33.8182 31)
-			(xy 33.80463 30.723768) (xy 33.76405 30.450196) (xy 33.69685 30.181919) (xy 33.603678 29.921521)
-			(xy 33.485431 29.671509) (xy 33.343248 29.434291) (xy 33.178499 29.212152) (xy 32.992769 29.007231)
-			(xy 32.787848 28.821501) (xy 32.565709 28.656752) (xy 32.328491 28.514569) (xy 32.078479 28.396322)
-			(xy 31.818081 28.30315) (xy 31.549804 28.23595) (xy 31.276232 28.19537) (xy 31 28.1818)
+			(xy 30.3912 33.6477) (xy 30.3848 33.5916) (xy 30.3476 33.4174) (xy 30.3104 33.243299) (xy 30.2732 33.0691)
+			(xy 30.2112 33.0691) (xy 30.1492 33.0691) (xy 30.0872 33.0691) (xy 30.0799 33.0342) (xy 30.0725 32.9992)
+			(xy 30.0652 32.9643) (xy 30.1272 32.9643) (xy 30.1892 32.9643) (xy 30.2512 32.9643) (xy 30.2349 32.8887)
+			(xy 30.2185 32.8132) (xy 30.202394 32.738595) (xy 30.097276 32.688879) (xy 29.936084 32.592264) (xy 29.785137 32.480315)
+			(xy 29.645891 32.354109) (xy 29.519685 32.214863) (xy 29.407736 32.063916) (xy 29.311121 31.902724)
+			(xy 29.230771 31.732838) (xy 29.16746 31.555895) (xy 29.121797 31.373597) (xy 29.094222 31.187702)
+			(xy 29.085 31) (xy 29.094222 30.812297) (xy 29.121797 30.626402) (xy 29.16746 30.444104) (xy 29.230771 30.267161)
+			(xy 29.311121 30.097275) (xy 29.407736 29.936083) (xy 29.519685 29.785136) (xy 29.645891 29.64589)
+			(xy 29.785137 29.519684) (xy 29.936084 29.407735) (xy 30.097276 29.31112) (xy 30.267162 29.23077)
+			(xy 30.444105 29.167459) (xy 30.626403 29.121796) (xy 30.812298 29.094221) (xy 31 29.085) (xy 31.187703 29.094221)
+			(xy 31.373598 29.121796) (xy 31.555896 29.167459) (xy 31.732839 29.23077) (xy 31.902725 29.31112)
+			(xy 32.063917 29.407735) (xy 32.214864 29.519684) (xy 32.35411 29.64589) (xy 32.480316 29.785136)
+			(xy 32.592265 29.936083) (xy 32.68888 30.097275) (xy 32.76923 30.267161) (xy 32.832541 30.444104)
+			(xy 32.878204 30.626402) (xy 32.905779 30.812297) (xy 32.915 31) (xy 32.905779 31.187702) (xy 32.878204 31.373597)
+			(xy 32.832541 31.555895) (xy 32.76923 31.732838) (xy 32.68888 31.902724) (xy 32.592265 32.063916)
+			(xy 32.480316 32.214863) (xy 32.35411 32.354109) (xy 32.214864 32.480315) (xy 32.063917 32.592264)
+			(xy 31.902725 32.688879) (xy 31.732839 32.769229) (xy 31.555896 32.83254) (xy 31.373598 32.878203)
+			(xy 31.187703 32.905778) (xy 31 32.915) (xy 30.812298 32.905778) (xy 30.626403 32.878203) (xy 30.444105 32.83254)
+			(xy 30.354434 32.800455) (xy 30.3662 32.8549) (xy 30.378 32.909599) (xy 30.3899 32.9643) (xy 30.4366 32.9643)
+			(xy 30.4834 32.9643) (xy 30.5302 32.9643) (xy 30.5375 32.9992) (xy 30.5449 33.0342) (xy 30.5522 33.0691)
+			(xy 30.5054 33.0691) (xy 30.4586 33.0691) (xy 30.4118 33.0691) (xy 30.4547 33.2715) (xy 30.4975 33.473799)
+			(xy 30.5404 33.6761) (xy 30.5375 33.7592) (xy 30.521922 33.774688) (xy 30.723769 33.804629) (xy 31 33.8182)
+			(xy 31.276232 33.804629) (xy 31.549804 33.764049) (xy 31.818081 33.696849) (xy 32.078479 33.603677)
+			(xy 32.328491 33.48543) (xy 32.565709 33.343247) (xy 32.787848 33.178498) (xy 32.992769 32.992768)
+			(xy 33.178499 32.787847) (xy 33.343248 32.565708) (xy 33.485431 32.32849) (xy 33.603678 32.078478)
+			(xy 33.69685 31.81808) (xy 33.76405 31.549803) (xy 33.80463 31.276231) (xy 33.8182 31) (xy 33.80463 30.723768)
+			(xy 33.76405 30.450196) (xy 33.69685 30.181919) (xy 33.603678 29.921521) (xy 33.485431 29.671509)
+			(xy 33.343248 29.434291) (xy 33.178499 29.212152) (xy 32.992769 29.007231) (xy 32.787848 28.821501)
+			(xy 32.565709 28.656752) (xy 32.328491 28.514569) (xy 32.078479 28.396322) (xy 31.818081 28.30315)
+			(xy 31.549804 28.23595) (xy 31.276232 28.19537) (xy 31 28.1818)
 		)
 		(stroke
